File: Z80_DualPIC.kicad_sch (KiCad schematic)
At the start: 38 parts, among them J1 ICSP, J2 UART, J3 I2C, J4 microSD, J5 DE15_Socket_HighDensity_Mount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, J6 M1_O, J7 USB_B_Mini, J8 Free_Pins, SW1 Slider_Switch, SW2 Z80_RESET, U1 Z84C00_PLCC, U2 PIC1-MMU, U3 AS6C4008-55PCN, U6 PIC2-IO-PROG, Y1 CXO_DIP8, Y2 Crystal

Commit message: finish routing & added README.md
Parts:
- D1: value LED-PWR -> PWR
- J4: footprint Connector_PinHeader_2.54mm:PinHeader_1x06_P2.54mm_Vertical -> Connector_PinSocket_2.54mm:PinSocket_1x06_P2.54mm_Vertical
- J5: value DE15_Socket_HighDensity_MountingHoles -> VGA-DB15
- J6: value M1_O -> M1
- J8: value Free_Pins -> FREE_PINS
- SW1: value Slider_Switch -> ON/OFF
- U1: value Z84C00_PLCC -> Z84C00/PLCC
- Y1: value CXO_DIP8 -> CANNED-DIP8
Changed lines of the file:
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@@
 			)
 		)
-		(property "Value" "Free_Pins"
+		(property "Value" "FREE_PINS"
 			(at 198.12 153.6699 0)
 			(show_name no)
@@
 			)
 		)
-		(property "Footprint" "Connector_PinHeader_2.54mm:PinHeader_1x06_P2.54mm_Vertical"
+		(property "Footprint" "Connector_PinSocket_2.54mm:PinSocket_1x06_P2.54mm_Vertical"
 			(at 269.24 149.86 0)
 			(hide yes)
@@
 			)
 		)
-		(property "Value" "DE15_Socket_HighDensity_MountingHoles"
+		(property "Value" "VGA-DB15"
 			(at 107.95 143.51 0)
 			(show_name no)
@@
 			)
 		)
-		(property "Value" "Slider_Switch"
+		(property "Value" "ON/OFF"
 			(at 220.98 109.22 0)
 			(show_name no)
@@
 			)
 		)
-		(property "Value" "M1_O"
+		(property "Value" "M1"
 			(at 38.1 105.4099 0)
 			(show_name no)
@@
 			)
 		)
-		(property "Value" "Z84C00_PLCC"
+		(property "Value" "Z84C00/PLCC"
 			(at 52.9433 24.13 0)
 			(show_name no)
@@
 			)
 		)
-		(property "Value" "CXO_DIP8"
-			(at 68.326 121.666 0)
+		(property "Value" "CANNED-DIP8"
+			(at 69.088 121.666 0)
 			(show_name no)
 			(do_not_autoplace no)
@@
 			)
 		)
-		(property "Value" "LED-PWR"
-			(at 39.878 171.704 0)
+		(property "Value" "PWR"
+			(at 40.386 170.18 0)
 			(show_name no)
 			(do_not_autoplace no)

Commit message: add IORQ, WR, RD & A0~A6 into PIC#2
Parts:
- removed J8: FREE_PINS, Connector_PinHeader_2.54mm:PinHeader_1x10_P2.54mm_Vertical, symbol Connector_Generic:Conn_01x10
- SW1: value ON/OFF -> ON|OFF
Connections:
- net RA0 is gone; now on net A0: U6.2 (RA0)
- net RA5 is gone; now on net A5: U6.7 (RA5)
- net RB5 is gone; now on net RED: U6.38 (RB5)
- net RC0 is gone; now on net VSYNC: U6.15 (RC0)
- net RC1 is gone; now on net HSYNC: U6.16 (RC1)
- net RC2 is gone; now on net SCK: U6.17 (RC2)
- net RC5 is gone; now on net CS: U6.24 (RC5)
- net RE0 is gone; now on net A6: U6.8 (RE0)
- net RE1 is gone; now on net MISO: U6.9 (RE1)
- net RE2 is gone; now on net MOSI: U6.10 (RE2)
- net A1: now also U6.3 (RA1)
- net A2: now also U6.4 (RA2)
- net A3: now also U6.5 (RA3)
- net A4: now also U6.6 (RA4)
- net BLUE: now also U6.36 (RB3); no longer U6.35 (RB2)
- net CS: no longer U6.3 (RA1)
- net GREEN: now also U6.37 (RB4); no longer U6.36 (RB3)
- net HSYNC: no longer U6.34 (RB1)
- net IORQ: now also U6.33 (RB0)
- net MISO: no longer U6.6 (RA4)
- net MOSI: no longer U6.5 (RA3)
- net RD: now also U6.34 (RB1)
- net RED: no longer U6.37 (RB4)
- net SCK: no longer U6.4 (RA2)
- net VSYNC: no longer U6.33 (RB0)
- net WR: now also U6.35 (RB2)

Commit message: add CLK to pulse Z80 clock + interrupt pins.
Parts:
- removed J6: M1, Connector_PinHeader_2.54mm:PinHeader_1x01_P2.54mm_Vertical, symbol Connector_Generic:Conn_01x01
- added D2: HALT, LED_THT:LED_D3.0mm, symbol Device:LED
- added R14: 330, Resistor_THT:R_Axial_DIN0207_L6.3mm_D2.5mm_P10.16mm_Horizontal, symbol Device:R
Connections:
- net A5: no longer U6.7 (RA5)
- net A6: no longer U6.8 (RE0)
- net GND: now also D1.1 (K); no longer R13.1
- net HALT: now also D2.1 (K); no longer U2.1 (RE3/~{MCLR})
- net INT: now also U6.7 (RA5); no longer U2.14 (RA6)
- net M1: now also U2.1 (RE3/~{MCLR}), U6.8 (RE0)
- net VCC: now also R13.2, R14.2; no longer D1.1 (K)
- net Z80_CLK: now also U2.14 (RA6)
- net at D1.2 (A): now also R13.1; no longer R13.2
- new net: D2.2 (A), R14.1
Other:
- note added: "Active-LOW : It must be tied High via a resistor to prevent random, unrecoverable system resets."
- note added: "Active-LOW: Need Pull-UP HIGH to Prevents Z80 glitching during PIC power-on boot phase."
- note added: "Active-LOW: Need Pull-UP HIGH to keeps Z80 running normally until PIC requests the bus."
- note added: "Active-LOW: Need to PUll-UP HIGH, As Active-Low to disable. Only need to wait for slow SRAM. AS6C4008 is 55ns too fast to wait."
- note added: "Active-LOW: Need to Pull-Up HIGH. To signal the Z80 when an SD card read finishes."
- note added: "Active-LOW: use it as a sink. CPU HALT -> 0V CPU EXEC -> 5V current = ~5mA"
- note added: "INTOSC clock 4xPLL, 32Mhz on FOSC/4 = 8Mhz"
- note added: "PIC#1 = MMU A Passive Extension, So it doesn't need INT-pin."
- note added: "PIC#2 Interrupt as Ex.Module : - Pull INT=LOW(0) -> Interupt Z80 - Send Vector Byte via (D0..D7) - Wait Z80 jump -> ISR Table: UART_PORT: IN A, (ADDRESS_LABEL) Listen for : IORQ+RD=LOW(0) && M1+WR=HIGH(1) => Match (A0..A4) with ADDRESS_LABEL -> Send a Byte back -> (D0..D7) => Release INT=HIGH(1)"
- note added: "Pull BUSREQ -> LOW to force Z80 release Address Bus & Copy ROM from microSD -> SRAM"
- note removed: "It must be tied High via a resistor to prevent random, unrecoverable system resets."
- note removed: "Need Pull-UP HIGH : Keeps Z80 running normally until PIC requests the bus."
- note removed: "Need Pull-UP HIGH : Prevents Z80 glitching during PIC power-on boot phase."
- note removed: "Need to PUll-UP HIGH, As Active-Low to disable. AS6C4008 is 55ns too fast to wait."
- note removed: "Need to Pull-Up HIGH. To signal the Z80 when an SD card read finishes."
- note removed: "Pull BUSREQ -> LOW to force Z80 release Address Bus and copy ROM from microSD -> SRAM"
- moved on the sheet: C4, C5, C6, C7, C8, J5, R10, R11, R12, R3, R4, R5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
